File: Proyecto.kicad_pcb (KiCad board)
At the start: 2 copper layers, 111.1 x 84.8 mm, 52 parts, among them P1 CONN_01X03, P2 CONN_01X03, Q1 BC808-40, Q2 BC808-40, U1 MCP2515, U2 MCP2551-I/SN, U3 AMS1117, U4 ACS712, U5 ACS712

Commit message: fix
Parts:
- moved PIN_R1 1.05 mm to (114.2, 61.8)
Routing:
- net /3.3V: track 8.82 -> 53.1 mm
- net GND: track 422.4 -> 446.8 mm, vias 5 -> 6
- net /R2: track 11.0 -> 22.6 mm
- net /AC2: track 43.2 -> 54.5 mm
- net /R1: track 4.67 -> 15.9 mm
- net /AC1: track 53.1 -> 64.0 mm
- net +5V: track 421.4 -> 429.9 mm
- net pin23: track 32.4 -> 33.2 mm
