File: Proyecto.kicad_pcb (KiCad board)
At the start: 2 copper layers, 101.7 x 64.5 mm, 54 parts, among them P1 CONN_01X03, P2 CONN_01X03, Q1 BC808-40, Q2 BC808-40, U1 MCP2515, U2 MCP2551-I/SN, U3 AMS1117, U4 ACS712, U5 ACS712, U6 AMS1117

Commit message: casa
Parts:
- added S3: CONN_01X03, Pin_Headers:Pin_Header_Straight_1x03, B.Cu at (114.9, 76.2)
- added S4: CONN_01X03, Pin_Headers:Pin_Header_Straight_1x03, B.Cu at (114.9, 79.8)
- PIN_L1, PIN_R1: footprint w_pin_strip:pin_socket_2mm_15 -> w_pin_strip:pin_socket_15
- moved D3 28.7 mm to (122.7, 108.8), turned to 90 degrees
- moved U6 5.11 mm to (101.6, 105.7)
- moved R4 4.98 mm to (114.3, 97.5), turned to 90 degrees
- moved S1 4.84 mm to (114.9, 69.1)
- moved S2 4.84 mm to (114.9, 72.6)
- moved D1 4.04 mm to (100.4, 51.8)
- moved R12 2.62 mm to (91.2, 103.9)
- moved PIN_L1 2.55 mm to (95.2, 85.1)
- moved PIN_R1 2.55 mm to (110.5, 85.1)
- moved Q2 2.44 mm to (118.0, 96.8), turned to 90 degrees
- moved C7 2.43 mm to (81.8, 53.4)
- moved R1 2.09 mm to (89.5, 59.7)
- moved R2 1.87 mm to (89.4, 56.3)
- moved C12 1.02 mm to (99.0, 95.1)
Connections:
- PIN_R1 pad 6: Net-(PIN_R1-Pad6) -> /PIN25
- PIN_R1 pad 7: Net-(PIN_R1-Pad7) -> /PIN26
Routing:
- net +5V: track 457.2 -> 427.0 mm, vias 2 -> 4
- net GND: track 486.2 -> 464.2 mm, vias 4 -> 2
- net Net-(D3-Pad2): track 34.8 -> 18.4 mm
- net /PIN26: track 0.00 -> 7.30 mm
- net +3.3V: track 27.7 -> 21.7 mm
- net /AC2: track 45.2 -> 39.5 mm
- net /CS: track 31.8 -> 37.0 mm
- net /SCK: track 59.7 -> 64.7 mm
- net /PIN23: track 5.01 -> 0.00 mm
- net /PIN24: track 4.88 -> 0.00 mm
- net /R1: track 8.06 -> 3.92 mm
- net /LED: track 10.7 -> 14.7 mm
- net Net-(ESP8266-Pad7): track 13.8 -> 10.4 mm
- net /AC1: track 47.2 -> 50.3 mm
- net Net-(R1-Pad2): track 12.6 -> 15.5 mm
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- removed copper zone on F.Cu, net GND

Commit message: full ok
Parts:
- moved Q1 4.21 mm to (130.4, 81.3)
- moved S1 2.54 mm to (115.1, 71.6)
- moved S4 2.54 mm to (115.1, 82.3)
- moved S2 2.54 mm to (115.1, 75.2)
- moved S3 2.54 mm to (115.1, 78.7)
- moved R3 1.50 mm to (129.3, 84.8)
Routing:
- net +5V: track 427.0 -> 459.2 mm, vias 4 -> 6
- net +3.3V: track 21.7 -> 35.2 mm
- net /AC1: track 50.3 -> 43.3 mm
- net Net-(ESP8266-Pad7): track 10.4 -> 16.6 mm
- net /PIN24: track 0.00 -> 5.94 mm
- net Net-(PIN_L1-Pad15): track 1.67 -> 7.21 mm
- net /PIN23: track 0.00 -> 5.52 mm
- net /PIN25: track 0.00 -> 5.10 mm
- net Net-(D2-Pad2): track 18.8 -> 14.3 mm
- net /PIN26: track 7.30 -> 4.68 mm
- net Net-(Q1-Pad1): track 6.30 -> 4.02 mm
- net /R2: track 16.9 -> 15.4 mm

Commit message: fix
Parts:
- added C13: 10uf, w_capacitors:CP_5x11mm, B.Cu at (95.5, 108.0)
- added C14: 10uf, w_capacitors:CP_5x11mm, B.Cu at (117.2, 61.2)
Routing:
- net GND: track 464.2 -> 470.0 mm
- net +3.3V: track 35.2 -> 36.7 mm
- net +5V: track 459.2 -> 460.2 mm
- added copper zone on F.Cu, net +5V
- added copper zone on F.Cu, net GND
