File: Proyecto.sch (KiCad schematic (older format))
At the start: 25 parts, among them IC1 ATMEGA328P-A, K1 HK4100F, Q1 BC808-40, SW1 SW_PUSH, U1 MCP2515, U2 MCP2551-I/SN, U3 AMS1117, U4 ACS712

Commit message: fix
Parts:
- added CFilter1, CFliter1: 1nf, Capacitors_SMD:C_1206, symbol C
- added D2: D, Diodes_ThroughHole:Diode_DO-35_SOD27_Horizontal_RM10, symbol D
- added K2: HK4100F, symbol HK4100F
- added P2: CONN_01X03, Terminal_Blocks:TerminalBlock_Pheonix_MPT-2.54mm_3pol, symbol CONN_01X03
- added Q2: BC808-40, TO_SOT_Packages_SMD:SOT-23, symbol BC808-40
- added R3: R, Resistors_SMD:R_1210_HandSoldering, symbol R
- added Serial1: CONN_01X02, Pin_Headers:Pin_Header_Straight_1x02, symbol CONN_01X02
- added U5: ACS712, SMD_Packages:SOIC-8-N, symbol ACS712
- CAN1: renamed from P?; footprint (none) -> Terminal_Blocks:TerminalBlock_Pheonix_MPT-2.54mm_2pol
- Carga1: renamed from P?; footprint (none) -> Pin_Headers:Pin_Header_Straight_1x02
- IC1: footprint TQFP32 -> Housings_QFP:TQFP-32_7x7mm_Pitch0.8mm
- P1: renamed from P?; footprint (none) -> Terminal_Blocks:TerminalBlock_Pheonix_MPT-2.54mm_3pol
- SW1: footprint (none) -> Buttons_Switches_ThroughHole:SW_PUSH_SMALL
- gave numbers to parts that had none: 1
Connections:
- net labels added: AC1, AC2
- wire segments 104 -> 159
Other:
- moved on the sheet: D1, P1, Q1, R2, U4

Commit message: add componenets
Parts:
- removed K1, K2: HK4100F, symbol HK4100F
- added C10, C11, C3, C4, C5, C6, C7: 100nf, Capacitors_SMD:C_1206_HandSoldering, symbol C
- added D1: 4007, Diodes_ThroughHole:Diode_DO-35_SOD27_Horizontal_RM10, symbol D
- added Relay1, Relay2: Songle_SRD, Relays_ThroughHole:Relay_SANYOU_SRD_Series_Form_C, symbol Songle_SRD
- added S0: CONN_01X02, Terminal_Blocks:TerminalBlock_Pheonix_MPT-2.54mm_2pol, symbol CONN_01X02
- 16Mhz1, Crystal1: footprint (none) -> Crystals:Crystal_HC49-U_Vertical
- C1: renamed from C2; value C -> 22pf
- C2: renamed from C1; value C -> 22pf
- C8: renamed from C3; footprint Capacitors_SMD:C_1210 -> Capacitors_SMD:C_1206_HandSoldering
- C9: renamed from C4; value C -> 22pf; footprint Capacitors_SMD:C_1210 -> Capacitors_SMD:C_1206_HandSoldering
- D2: renamed from D1; value D -> 1N4001
- D3: renamed from D2; value D -> 1N4001
- U1: footprint MODULE -> Housings_SOIC:SOIC-18_7.5x11.6mm_Pitch1.27mm
Connections:
- net labels removed: VCC
- wire segments 159 -> 189
- no-connect marks 7 -> 17
Other:
- moved on the sheet: S1, S2

Commit message: fix
se quito el micro y se coloco pines hembra para insertar NanoArduino en
placa
Parts:
- removed 16Mhz1: Crystal, Crystals:Crystal_HC49-U_Vertical, symbol Crystal
- removed C1, C2: 22pf, Capacitors_SMD:C_1210, symbol C
- removed C5: 100nf, Capacitors_SMD:C_1206_HandSoldering, symbol C
- removed IC1: ATMEGA328P-A, Housings_QFP:TQFP-32_7x7mm_Pitch0.8mm, symbol ATMEGA328P-A
- removed R1: R, Resistors_SMD:R_1206_HandSoldering, symbol R
- removed R4: 120, Resistors_SMD:R_1210_HandSoldering, symbol R
- removed SW1: SW_PUSH, Buttons_Switches_ThroughHole:SW_PUSH_SMALL, symbol SW_PUSH
- added D_RX1, D_TX1, LED_BLINK1: LED, LEDs:LED-5MM, symbol LED
- added PIN_L1, PIN_R1: CONN_01X15, Pin_Headers:Pin_Header_Straight_1x15, symbol CONN_01X15
- added R10, R8, R9: 1k, Resistors_ThroughHole:Resistor_Horizontal_RM10mm, symbol R
- added R5: 120, Resistors_ThroughHole:Resistor_Horizontal_RM10mm, symbol R
- C10, C11, C3, C4, C6, C7, C8, C9: footprint Capacitors_SMD:C_1206_HandSoldering -> Capacitors_ThroughHole:C_Disc_D3_P2.5
- CFilter1, CFliter1: footprint Capacitors_SMD:C_1206 -> Capacitors_ThroughHole:C_Disc_D3_P2.5
- Crystal2: renamed from Crystal1; value 16mhz -> 16Mhz
- R1: renamed from 10k1; value R -> 10k; footprint Resistors_SMD:R_1210 -> Resistors_ThroughHole:Resistor_Horizontal_RM15mm
- R2: renamed from 10k2; value R -> 10k; footprint Resistors_SMD:R_1210 -> Resistors_ThroughHole:Resistor_Horizontal_RM10mm
- R3: renamed from R2; value R -> 1k; footprint Resistors_SMD:R_1210_HandSoldering -> Resistors_ThroughHole:Resistor_Horizontal_RM10mm
- R4: renamed from R3; value R -> 1k; footprint Resistors_SMD:R_1210_HandSoldering -> Resistors_ThroughHole:Resistor_Horizontal_RM10mm
Connections:
- net labels added: CS, INT, LED_BLINK, R1, R2, SCK, SI, SO
- net labels removed: RESET
- wire segments 189 -> 165
- no-connect marks 17 -> 21
Other:
- moved on the sheet: C10, C11, C4, CFilter1, D2, P1, Q1, R3, Relay1, Serial1, U4

Commit message: fix terrena
Parts:
- added D4: LED 2, LEDs:LED-5MM, symbol LED
- added R11: 1k, Resistors_ThroughHole:Resistor_Horizontal_RM10mm, symbol R
- R1: footprint Resistors_ThroughHole:Resistor_Horizontal_RM15mm -> Resistors_ThroughHole:Resistor_Horizontal_RM10mm
- U2: footprint Power_Integrations:SO-8 -> SMD_Packages:SOIC-8-N
Connections:
- net labels added: LED, rx, tx
- net labels removed: LED_BLINK
- wire segments 165 -> 171
- no-connect marks 21 -> 20
Other:
- moved on the sheet: PIN_R1, Serial1

Commit message: fix
Parts:
- added U6: MCP2515, Housings_SOIC:SOIC-18_7.5x11.6mm_Pitch1.27mm, symbol MCP2515
Connections:
- wire segments 171 -> 176
- no-connect marks 20 -> 39
Other:
- moved on the sheet: Relay1

Commit message: fix casa
se dieron vuelta los pines del nano arudino
Parts:
- removed U6: MCP2515, Housings_SOIC:SOIC-18_7.5x11.6mm_Pitch1.27mm, symbol MCP2515
- U1: symbol MCP2515 -> MCP2515-RESCUE-Proyecto
Connections:
- wire segments 176 -> 175
- no-connect marks 39 -> 22
Changed lines of the file:
@@
 EESchema Schematic File Version 2
+LIBS:Proyecto-rescue
 LIBS:power
 LIBS:device
@@
 LIBS:mylib
 LIBS:HK4100F
-LIBS:acs712
-LIBS:AMS1117
 LIBS:Proyecto-cache
 EELAYER 25 0
@@
 $EndComp
 $Comp
-L MCP2515 U1
+L MCP2515-RESCUE-Proyecto U1
 U 1 1 576AE893
 P 4950 2700
@@
 NoConn ~ 1900 5200
 NoConn ~ 8950 3850
-$Comp
-L MCP2515 U6
-U 1 1 577574D8
-P 9300 2000
-F 0 "U6" H 9300 1900 50  0000 C CNN
-F 1 "MCP2515" H 9300 2100 50  0000 C CNN
-F 2 "Housings_SOIC:SOIC-18_7.5x11.6mm_Pitch1.27mm" H 9300 2000 50  0001 C CNN
-F 3 "DOCUMENTATION" H 9300 2000 50  0001 C CNN
-	1    9300 2000
-	1    0    0    -1
-$EndComp
-NoConn ~ 10050 1600
-NoConn ~ 10050 1700
-NoConn ~ 10050 1800
-NoConn ~ 10050 1900
-NoConn ~ 10050 2000
-NoConn ~ 10050 2100
-NoConn ~ 10050 2200
-NoConn ~ 10050 2300
-NoConn ~ 10050 2400
-NoConn ~ 8550 1600
-NoConn ~ 8550 1700
-NoConn ~ 8550 1800
-NoConn ~ 8550 1900
-NoConn ~ 8550 2000
-NoConn ~ 8550 2100
-NoConn ~ 8550 2200
-NoConn ~ 8550 2300
-$Comp
-L GND #PWR?
-U 1 1 57758B22
-P 8550 2500
-F 0 "#PWR?" H 8550 2250 50  0001 C CNN
-F 1 "GND" H 8550 2350 50  0000 C CNN
-F 2 "" H 8550 2500 50  0000 C CNN
-F 3 "" H 8550 2500 50  0000 C CNN
-	1    8550 2500
-	1    0    0    -1
-$EndComp
-Wire Wire Line
-	8550 2500 8550 2400
 $EndSCHEMATC

Commit message: fix terrena
Parts:
- removed Serial1: CONN_01X02, Pin_Headers:Pin_Header_Straight_1x02, symbol CONN_01X02
- added ESP8266: CONN_02X04, Pin_Headers:Pin_Header_Straight_2x04, symbol CONN_02X04
- added LED_Gp1, LED_Gp2: LED, LEDs:LED-5MM, symbol LED
- added R12, R6, R7: 1k, Resistors_ThroughHole:Resistor_Horizontal_RM10mm, symbol R
- added R13: 2k2, Resistors_ThroughHole:Resistor_Horizontal_RM10mm, symbol R
- LED_Vcc1: renamed from D4; value LED 2 -> LED
- renumbered LED_BLINK1 to LED1
Connections:
- net labels added: 3.3V, Gp1, Gp2, Vcc
- net labels removed: rx, tx
- wire segments 175 -> 200
- no-connect marks 22 -> 21
Other:
- moved on the sheet: LED1, LED_Vcc1, R10, R11

Commit message: fix
Parts:
- CAN1, Carga1, S0: symbol CONN_01X02 -> CONN_01X02-RESCUE-Proyecto
Changed lines of the file:
@@
 EESchema Schematic File Version 2
+LIBS:Proyecto-rescue
 LIBS:power
 LIBS:device
@@
 LIBS:contrib
 LIBS:valves
-LIBS:MCP2515 E
-LIBS:SongleRelay
-LIBS:mylib
-LIBS:HK4100F
-LIBS:acs712
-LIBS:AMS1117
 LIBS:Proyecto-cache
 EELAYER 25 0
@@
 $EndComp
 $Comp
-L CONN_01X02 CAN1
+L CONN_01X02-RESCUE-Proyecto CAN1
 U 1 1 576B8DD1
 P 8350 3200
@@
 $EndComp
 $Comp
-L CONN_01X02 Carga1
+L CONN_01X02-RESCUE-Proyecto Carga1
 U 1 1 576B90D8
 P 8000 2550
@@
 $EndComp
 $Comp
-L CONN_01X02 S0
+L CONN_01X02-RESCUE-Proyecto S0
 U 1 1 576D275D
 P 700 1350
